File: pcb/modelh.sch (KiCad schematic (older format))
At the start: 46 parts, among them J1 USB_B, J2 Conn_01x16, J3 Conn_01x12, J4 Conn_01x04, J5 Conn_02x03_Odd_Even, J6 Conn_02x05_Odd_Even, J7 Conn_01x05, J8 Conn_01x05, J9 Conn_01x05, SW1 SW_Push, U1 STM32F103C8Tx, U2 AMS1117-3.3, Y1 8MHz

Commit message: WIPWIP
Parts:
- R1, R2: LCSC C21190 -> C23138
- R7, R8, R9: value 60 -> 100
Changed lines of the file:
@@
 P 8900 4600
 F 0 "R7" V 8850 4750 50  0000 C CNN
-F 1 "60" V 8900 4600 50  0000 C CNN
+F 1 "100" V 8900 4600 50  0000 C CNN
 F 2 "Resistor_SMD:R_0805_2012Metric" V 8830 4600 50  0001 C CNN
 F 3 "~" H 8900 4600 50  0001 C CNN
@@
 P 8900 4700
 F 0 "R8" V 8850 4850 50  0000 C CNN
-F 1 "60" V 8900 4700 50  0000 C CNN
+F 1 "100" V 8900 4700 50  0000 C CNN
 F 2 "Resistor_SMD:R_0805_2012Metric" V 8830 4700 50  0001 C CNN
 F 3 "~" H 8900 4700 50  0001 C CNN
@@
 P 8900 4900
 F 0 "R9" V 8850 5050 50  0000 C CNN
-F 1 "60" V 8900 4900 50  0000 C CNN
+F 1 "100" V 8900 4900 50  0000 C CNN
 F 2 "Resistor_SMD:R_0805_2012Metric" V 8830 4900 50  0001 C CNN
 F 3 "~" H 8900 4900 50  0001 C CNN
@@
 F 2 "Resistor_SMD:R_0603_1608Metric" V 830 6600 50  0001 C CNN
 F 3 "~" H 900 6600 50  0001 C CNN
-F 4 "C21190" H 900 6600 50  0001 C CNN "LCSC"
+F 4 "C23138" H 900 6600 50  0001 C CNN "LCSC"
 	1    900  6600
 	1    0    0    -1
@@
 F 2 "Resistor_SMD:R_0603_1608Metric" V 1380 6600 50  0001 C CNN
 F 3 "~" H 1450 6600 50  0001 C CNN
-F 4 "C21190" H 1450 6600 50  0001 C CNN "LCSC"
+F 4 "C23138" H 1450 6600 50  0001 C CNN "LCSC"
 	1    1450 6600
 	1    0    0    -1
@@
 Wire Wire Line
 	2550 1400 2100 1400
-$Comp
-L Device:R R16
-U 1 1 5F9EF12F
-P 1950 1100
-F 0 "R16" V 1743 1100 50  0000 C CNN
-F 1 "0" V 1834 1100 50  0000 C CNN
-F 2 "Resistor_SMD:R_0805_2012Metric_Pad1.15x1.40mm_HandSolder" V 1880 1100 50  0001 C CNN
-F 3 "~" H 1950 1100 50  0001 C CNN
-F 4 "C17477" H 1950 1100 50  0001 C CNN "LCSC"
-	1    1950 1100
-	0    1    1    0
-$EndComp
 Wire Wire Line
 	4900 2800 5100 2800
@@
 Wire Wire Line
 	8950 6050 9450 6050
+$Comp
+L Device:R R16
+U 1 1 5F9EF12F
+P 1950 1100
+F 0 "R16" V 1743 1100 50  0000 C CNN
+F 1 "0" V 1834 1100 50  0000 C CNN
+F 2 "Resistor_SMD:R_0805_2012Metric_Pad1.15x1.40mm_HandSolder" V 1880 1100 50  0001 C CNN
+F 3 "~" H 1950 1100 50  0001 C CNN
+F 4 "C17477" H 1950 1100 50  0001 C CNN "LCSC"
+	1    1950 1100
+	0    1    1    0
+$EndComp
 $EndSCHEMATC

Commit message: Finish footprints
Parts:
- J2: footprint Connector_PinSocket_2.54mm:PinSocket_1x16_P2.54mm_Vertical -> modelh:ModelH-triomate-cols16
- J3: footprint Connector_PinSocket_2.54mm:PinSocket_1x12_P2.54mm_Vertical -> modelh:ModelH-triomate-rows12
- J4: footprint Connector_PinSocket_2.54mm:PinSocket_1x04_P2.54mm_Vertical -> modelh:ModelH-tripmate-leds4
Changed lines of the file:
@@
 F 0 "J2" H 10380 1942 50  0000 L CNN
 F 1 "Conn_01x16" H 10380 1851 50  0000 L CNN
-F 2 "Connector_PinSocket_2.54mm:PinSocket_1x16_P2.54mm_Vertical" H 10300 1950 50  0001 C CNN
+F 2 "modelh:ModelH-triomate-cols16" H 10300 1950 50  0001 C CNN
 F 3 "~" H 10300 1950 50  0001 C CNN
 	1    10300 1950
@@
 F 0 "J4" H 10380 4692 50  0000 L CNN
 F 1 "Conn_01x04" H 10380 4601 50  0000 L CNN
-F 2 "Connector_PinSocket_2.54mm:PinSocket_1x04_P2.54mm_Vertical" H 10300 4700 50  0001 C CNN
+F 2 "modelh:ModelH-tripmate-leds4" H 10300 4700 50  0001 C CNN
 F 3 "~" H 10300 4700 50  0001 C CNN
 	1    10300 4700
@@
 F 0 "J3" H 10380 3692 50  0000 L CNN
 F 1 "Conn_01x12" H 10380 3601 50  0000 L CNN
-F 2 "Connector_PinSocket_2.54mm:PinSocket_1x12_P2.54mm_Vertical" H 10300 3700 50  0001 C CNN
+F 2 "modelh:ModelH-triomate-rows12" H 10300 3700 50  0001 C CNN
 F 3 "~" H 10300 3700 50  0001 C CNN
 	1    10300 3700
