File: pcb/modelh.kicad_pcb (KiCad board)
At the start: 2 copper layers, 150 x 38 mm, 50 parts, among them J1 USB_B, J2 Conn_01x16, J3 Conn_01x12, J4 Conn_01x04, J5 Conn_02x03_Odd_Even, J6 Conn_02x05_Odd_Even, J7 Conn_01x05, J8 Conn_01x05, J9 Conn_01x05, SW1 SW_Push, U1 STM32F103C8Tx, U2 AMS1117-3.3, Y1 8MHz

Commit message: WIP
Parts:
- moved J7 1.99 mm to (204.2, 67.9)
- moved J8 1.99 mm to (196.4, 67.9)
- moved J9 1.99 mm to (200.1, 67.9)
Routing:
- net +3V3: track 243.4 -> 246.1 mm, vias 3 -> 4
- net led2: track 98.0 -> 98.5 mm
- net GND: vias 28 -> 24
Changed lines of the file:
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@@
     (thickness 1.6)
     (drawings 30)
-    (tracks 577)
+    (tracks 579)
     (zones 0)
     (modules 50)
@@
     (pad_to_mask_clearance 0.0508)
     (solder_mask_min_width 0.101)
-    (aux_axis_origin 88.77 46.99)
-    (grid_origin 115.77 54.74)
+    (aux_axis_origin 64.77 46.99)
+    (grid_origin 64.77 46.99)
     (visible_elements FFFFFF7F)
     (pcbplotparams
@@
   )
   (module Connector_PinSocket_2.54mm:Conn_Generic_01x05 (layer F.Cu)
-    (at 196.97 66.04)
+    (at 196.37 67.94)
     (descr "Through hole straight socket strip, 1x05, 2.54mm pitch, single row (from Kicad 4.0.7), script generated")
     (tags "Through hole socket strip THT 1x05 2.54mm single row")
@@
   )
   (module Connector_PinSocket_2.54mm:Conn_Generic_01x05 (layer F.Cu)
-    (at 200.67 66.04)
+    (at 200.07 67.94)
     (descr "Through hole straight socket strip, 1x05, 2.54mm pitch, single row (from Kicad 4.0.7), script generated")
     (tags "Through hole socket strip THT 1x05 2.54mm single row")
@@
   )
   (module Connector_PinSocket_2.54mm:Conn_Generic_01x05 (layer F.Cu)
-    (at 204.77 66.04)
+    (at 204.17 67.94)
     (descr "Through hole straight socket strip, 1x05, 2.54mm pitch, single row (from Kicad 4.0.7), script generated")
     (tags "Through hole socket strip THT 1x05 2.54mm single row")
@@
     (tags resistor)
     (attr smd)
-    (fp_text reference R11 (at 0 -1.43) (layer F.SilkS)
+    (fp_text reference R11 (at 0 -1.43) (layer F.Fab)
       (effects (font (size 1 1) (thickness 0.15)))
     )
@@
     (effects (font (size 1 1) (thickness 0.15)))
   )
-  (gr_text GND (at 193.07 76.44) (layer F.SilkS)
+  (gr_text GND (at 192.77 78.19) (layer F.SilkS)
     (effects (font (size 1 1) (thickness 0.15)))
   )
-  (gr_text 3.3V (at 193.17 73.94) (layer F.SilkS)
+  (gr_text 3.3V (at 192.67 75.64) (layer F.SilkS)
     (effects (font (size 1 1) (thickness 0.15)))
   )
-  (gr_text LED2 (at 193.17 71.44) (layer F.SilkS)
+  (gr_text LED2 (at 192.62 73.04) (layer F.SilkS)
     (effects (font (size 1 1) (thickness 0.15)))
   )
-  (gr_text LED1 (at 193.17 68.84) (layer F.SilkS)
+  (gr_text LED1 (at 192.67 70.49) (layer F.SilkS)
     (effects (font (size 1 1) (thickness 0.15)))
   )
-  (gr_text LED0 (at 193.17 66.44) (layer F.SilkS)
+  (gr_text LED0 (at 192.67 67.94) (layer F.SilkS)
     (effects (font (size 1 1) (thickness 0.15)))
   )
@@
     (effects (font (size 1.5 1.5) (thickness 0.3)) (justify left))
   )
-  (gr_text Reset (at 97.37 75.24) (layer F.SilkS)
+  (gr_text Reset (at 106.42 79.69) (layer F.SilkS)
     (effects (font (size 1.5 1.5) (thickness 0.3)) (justify left))
   )
@@
   (segment (start 106.917658 67.524322) (end 105.385 69.05698) (width 0.25) (layer F.Cu) (net 1))
   (segment (start 105.21499 69.41001) (end 105.385 69.24) (width 0.5) (layer F.Cu) (net 1))
-  (via (at 107.27 82.24) (size 0.8) (drill 0.4) (layers F.Cu B.Cu) (net 1))
-  (via (at 107.27 81.24) (size 0.8) (drill 0.4) (layers F.Cu B.Cu) (net 1))
-  (via (at 107.27 80.24) (size 0.8) (drill 0.4) (layers F.Cu B.Cu) (net 1))
-  (via (at 107.27 79.24) (size 0.8) (drill 0.4) (layers F.Cu B.Cu) (net 1))
   (segment (start 112.6275 66.39292) (end 112.57229 66.33771) (width 0.5) (layer F.Cu) (net 1))
   (segment (start 112.6275 66.5775) (end 112.6275 66.39292) (width 0.5) (layer F.Cu) (net 1))
@@
   (segment (start 114.67 65.44) (end 111.67 65.44) (width 0.8) (layer B.Cu) (net 9))
   (segment (start 109.37 67.74) (end 109.37 69.14) (width 0.8) (layer B.Cu) (net 9))
-  (segment (start 114.67 65.44) (end 118.97 65.44) (width 0.8) (layer F.Cu) (net 9))
   (segment (start 119.770001 66.240001) (end 120.109999 66.240001) (width 0.8) (layer F.Cu) (net 9))
   (segment (start 118.97 65.44) (end 119.770001 66.240001) (width 0.8) (layer F.Cu) (net 9))
@@
   (segment (start 76.2825 60.215) (end 75.51999 60.97751) (width 0.25) (layer F.Cu) (net 9))
   (segment (start 76.2825 59.74) (end 76.2825 60.215) (width 0.25) (layer F.Cu) (net 9))
-  (segment (start 193.37 69.93) (end 197.03 73.59) (width 0.8) (layer F.Cu) (net 9))
-  (segment (start 193.37 66.24) (end 193.37 69.93) (width 0.8) (layer F.Cu) (net 9))
+  (segment (start 193.37 72.56) (end 196.37 75.56) (width 0.8) (layer F.Cu) (net 9))
+  (segment (start 193.37 66.24) (end 193.37 72.56) (width 0.8) (layer F.Cu) (net 9))
+  (segment (start 115.72 65.44) (end 118.97 65.44) (width 0.8) (layer F.Cu) (net 9))
+  (via (at 115.72 65.44) (size 0.8) (drill 0.4) (layers F.Cu B.Cu) (net 9))
+  (segment (start 115.72 65.44) (end 114.67 65.44) (width 0.8) (layer B.Cu) (net 9))
+  (segment (start 109.37 70.14) (end 109.37 69.14) (width 0.8) (layer B.Cu) (net 9))
   (segment (start 102.4075 73.2025) (end 102.77 73.2025) (width 0.25) (layer F.Cu) (net 10))
   (segment (start 100.97 74.64) (end 102.4075 73.2025) (width 0.25) (layer F.Cu) (net 10))
@@
   (segment (start 187.69 60.42) (end 187.74 60.42) (width 0.25) (layer F.Cu) (net 46))
   (segment (start 187.74 60.42) (end 188.59 60.42) (width 0.25) (layer F.Cu) (net 46))
+  (segment (start 188.59 60.42) (end 188.59 60.42) (width 0.25) (layer F.Cu) (net 46))
   (segment (start 188.59 60.42) (end 190.0125 60.42) (width 0.25) (layer F.Cu) (net 46))
   (via (at 188.59 60.42) (size 0.8) (drill 0.4) (layers F.Cu B.Cu) (net 46))
-  (segment (start 194.21 66.04) (end 197.02 66.04) (width 0.25) (layer B.Cu) (net 46))
-  (segment (start 188.59 60.42) (end 194.21 66.04) (width 0.25) (layer B.Cu) (net 46))
+  (segment (start 196.11 67.94) (end 196.37 67.94) (width 0.25) (layer B.Cu) (net 46))
+  (segment (start 188.59 60.42) (end 196.11 67.94) (width 0.25) (layer B.Cu) (net 46))
   (via (at 108.07 65.54) (size 0.6) (drill 0.3) (layers F.Cu B.Cu) (net 47))
   (via (at 121.27 65.34) (size 0.6) (drill 0.3) (layers F.Cu B.Cu) (net 47))
@@
   (segment (start 188.115 62.47) (end 188.54 62.47) (width 0.25) (layer F.Cu) (net 47))
   (segment (start 185.93982 64.64518) (end 188.115 62.47) (width 0.25) (layer F.Cu) (net 47))
+  (segment (start 188.54 62.47) (end 188.54 62.47) (width 0.25) (layer F.Cu) (net 47))
   (segment (start 188.54 62.47) (end 189.8625 62.47) (width 0.25) (layer F.Cu) (net 47))
   (via (at 188.54 62.47) (size 0.8) (drill 0.4) (layers F.Cu B.Cu) (net 47))
-  (segment (start 194.66 68.59) (end 197.03 68.59) (width 0.25) (layer B.Cu) (net 47))
-  (segment (start 188.54 62.47) (end 194.66 68.59) (width 0.25) (layer B.Cu) (net 47))
+  (segment (start 196.37 70.3) (end 196.37 70.48) (width 0.25) (layer B.Cu) (net 47))
+  (segment (start 188.54 62.47) (end 196.37 70.3) (width 0.25) (layer B.Cu) (net 47))
   (via (at 107.27 65.54) (size 0.6) (drill 0.3) (layers F.Cu B.Cu) (net 48))
   (segment (start 106.073554 65.54) (end 107.27 65.54) (width 0.25) (layer F.Cu) (net 48))
@@
   (segment (start 188.17 64.54) (end 188.57 64.54) (width 0.25) (layer F.Cu) (net 48))
   (segment (start 122.07 65.34) (end 122.494264 65.34) (width 0.25) (layer F.Cu) (net 48))
+  (segment (start 188.57 64.54) (end 188.57 64.54) (width 0.25) (layer F.Cu) (net 48))
   (segment (start 188.57 64.54) (end 189.8625 64.54) (width 0.25) (layer F.Cu) (net 48))
   (via (at 188.57 64.54) (size 0.8) (drill 0.4) (layers F.Cu B.Cu) (net 48))
-  (segment (start 195.17 71.14) (end 197.02 71.14) (width 0.25) (layer B.Cu) (net 48))
-  (segment (start 188.57 64.54) (end 195.17 71.14) (width 0.25) (layer B.Cu) (net 48))
+  (segment (start 188.57 65.22) (end 196.37 73.02) (width 0.25) (layer B.Cu) (net 48))
+  (segment (start 188.57 64.54) (end 188.57 65.22) (width 0.25) (layer B.Cu) (net 48))
   (segment (start 107.047363 60.465001) (end 109.769679 60.465001) (width 0.25) (layer F.Cu) (net 49))
   (segment (start 110.683002 59.551678) (end 110.683002 59.516338) (width 0.25) (layer F.Cu) (net 49))
@@
   (segment (start 87.47 59.065) (end 85.295 61.24) (width 1) (layer F.Cu) (net 54))
   (segment (start 87.47 57.49) (end 87.47 59.065) (width 1) (layer F.Cu) (net 54))
-  (segment (start 204.76 76.19) (end 204.77 76.2) (width 0.8) (layer F.Cu) (net 55))
-  (segment (start 200.66 76.19) (end 204.76 76.19) (width 0.8) (layer F.Cu) (net 55))
-  (segment (start 204.7 73.59) (end 204.77 73.66) (width 0.8) (layer F.Cu) (net 56))
-  (segment (start 200.67 73.59) (end 204.7 73.59) (width 0.8) (layer F.Cu) (net 56))
-  (segment (start 204.75 71.14) (end 204.77 71.12) (width 0.8) (layer F.Cu) (net 57))
-  (segment (start 200.66 71.14) (end 204.75 71.14) (width 0.8) (layer F.Cu) (net 57))
-  (segment (start 204.76 68.59) (end 204.77 68.58) (width 0.8) (layer F.Cu) (net 58))
-  (segment (start 200.67 68.59) (end 204.76 68.59) (width 0.8) (layer F.Cu) (net 58))
-  (segment (start 200.66 66.04) (end 204.77 66.04) (width 0.8) (layer F.Cu) (net 59))
+  (segment (start 204.16 78.09) (end 204.17 78.1) (width 0.8) (layer F.Cu) (net 55))
+  (segment (start 200.06 78.09) (end 204.16 78.09) (width 0.8) (layer F.Cu) (net 55))
+  (segment (start 204.1 75.49) (end 204.17 75.56) (width 0.8) (layer F.Cu) (net 56))
+  (segment (start 200.07 75.49) (end 204.1 75.49) (width 0.8) (layer F.Cu) (net 56))
+  (segment (start 204.15 73.04) (end 204.17 73.02) (width 0.8) (layer F.Cu) (net 57))
+  (segment (start 200.06 73.04) (end 204.15 73.04) (width 0.8) (layer F.Cu) (net 57))
+  (segment (start 204.16 70.49) (end 204.17 70.48) (width 0.8) (layer F.Cu) (net 58))
+  (segment (start 200.07 70.49) (end 204.16 70.49) (width 0.8) (layer F.Cu) (net 58))
+  (segment (start 200.06 67.94) (end 204.17 67.94) (width 0.8) (layer F.Cu) (net 59))
   (zone (net 1) (net_name GND) (layer F.Cu) (hatch edge 0.508)
     (connect_pads yes (clearance 0.5))

Commit message: WIP
Parts:
- C10, C11, C12, C13, C14: value 100 nF -> 100nF
- C9: footprint Capacitor_SMD:C_0603_1608Metric -> Capacitor_SMD:C_0402_1005Metric
- J7, J8, J9: footprint Connector_PinSocket_2.54mm:Conn_Generic_01x05 -> Connector_PinSocket_2.54mm:PinSocket_1x05_P2.54mm_Vertical
- R10, R5: value 1k -> 1.5k
- moved SW1 1.19 mm to (100.9, 80.3)
- moved C9 0.56 mm to (99.5, 73.4)
Routing:
- net nRST: track 40.4 -> 45.9 mm
